File: RP2040-Radio-Panel.kicad_pcb (KiCad board)
At the start: 2 copper layers, 14 x 18.4 mm, 1 part, among them U1 DM13A

Commit message: Add RP2040
Parts:
- removed U1: DM13A, Package_SO:SSOP-24_3.9x8.7mm_P0.635mm
Other:
- board outline removed
Changed lines of the file:
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@@
     )
   )
+  (property "DATE" "")
+  (property "KICAD6_USER_COMPONENTS_DIR" "${KIPRJMOD}/KiCad6-Components")
+  (property "VERSION" "")
   (net 0 "")
-  (net 1 "unconnected-(U1-GND-Pad1)")
-  (net 2 "unconnected-(U1-DIN-Pad2)")
-  (net 3 "unconnected-(U1-CLOCK-Pad3)")
-  (net 4 "unconnected-(U1-LATCH-Pad4)")
-  (net 5 "unconnected-(U1-OUT0-Pad5)")
-  (net 6 "unconnected-(U1-OUT1-Pad6)")
-  (net 7 "unconnected-(U1-OUT2-Pad7)")
-  (net 8 "unconnected-(U1-OUT3-Pad8)")
-  (net 9 "unconnected-(U1-OUT4-Pad9)")
-  (net 10 "unconnected-(U1-OUT5-Pad10)")
-  (net 11 "unconnected-(U1-OUT6-Pad11)")
-  (net 12 "unconnected-(U1-OUT7-Pad12)")
-  (net 13 "unconnected-(U1-OUT8-Pad13)")
-  (net 14 "unconnected-(U1-OUT9-Pad14)")
-  (net 15 "unconnected-(U1-OUT10-Pad15)")
-  (net 16 "unconnected-(U1-OUT11-Pad16)")
-  (net 17 "unconnected-(U1-OUT12-Pad17)")
-  (net 18 "unconnected-(U1-OUT13-Pad18)")
-  (net 19 "unconnected-(U1-OUT14-Pad19)")
-  (net 20 "unconnected-(U1-OUT15-Pad20)")
-  (net 21 "unconnected-(U1-~{EN}-Pad21)")
-  (net 22 "unconnected-(U1-DOUT-Pad22)")
-  (net 23 "unconnected-(U1-REXT-Pad23)")
-  (net 24 "unconnected-(U1-VDD-Pad24)")
-  (footprint "Package_SO:SSOP-24_3.9x8.7mm_P0.635mm" (layer "F.Cu")
-    (at 92.015 77.7875)
-    (descr "SSOP24: plastic shrink small outline package; 24 leads; body width 3.9 mm; lead pitch 0.635; (see NXP SSOP-TSSOP-VSO-REFLOW.pdf and sot556-1_po.pdf)")
-    (tags "SSOP 0.635")
-    (property "Sheetfile" "RP2040-Radio-Panel.kicad_sch")
-    (property "Sheetname" "")
-    (property "ki_description" "15-bit constant current LED driver")
-    (attr smd)
-    (fp_text reference "U1" (at 0 -5.4) (layer "F.SilkS")
-        (effects (font (size 1 1) (thickness 0.15)))
-    )
-    (fp_text value "DM13A" (at 0 5.4) (layer "F.Fab")
-        (effects (font (size 1 1) (thickness 0.15)))
-    )
-    (fp_text user "${REFERENCE}" (at 0 0) (layer "F.Fab")
-        (effects (font (size 0.8 0.8) (thickness 0.15)))
-    )
-    (fp_line (start -2.075 -4.475) (end -2.075 -4)
-      (stroke (width 0.15) (type solid)) (layer "F.SilkS"))
-    (fp_line (start -2.075 -4.475) (end 2.075 -4.475)
-      (stroke (width 0.15) (type solid)) (layer "F.SilkS"))
-    (fp_line (start -2.075 -4) (end -3.2 -4)
-      (stroke (width 0.15) (type solid)) (layer "F.SilkS"))
-    (fp_line (start -2.075 4.475) (end -2.075 3.9175)
-      (stroke (width 0.15) (type solid)) (layer "F.SilkS"))
-    (fp_line (start -2.075 4.475) (end 2.075 4.475)
-      (stroke (width 0.15) (type solid)) (layer "F.SilkS"))
-    (fp_line (start 2.075 -4.475) (end 2.075 -3.9175)
-      (stroke (width 0.15) (type solid)) (layer "F.SilkS"))
-    (fp_line (start 2.075 4.475) (end 2.075 3.9175)
-      (stroke (width 0.15) (type solid)) (layer "F.SilkS"))
-    (fp_line (start -3.45 -4.65) (end -3.45 4.65)
-      (stroke (width 0.05) (type solid)) (layer "F.CrtYd"))
-    (fp_line (start -3.45 -4.65) (end 3.45 -4.65)
-      (stroke (width 0.05) (type solid)) (layer "F.CrtYd"))
-    (fp_line (start -3.45 4.65) (end 3.45 4.65)
-      (stroke (width 0.05) (type solid)) (layer "F.CrtYd"))
-    (fp_line (start 3.45 -4.65) (end 3.45 4.65)
-      (stroke (width 0.05) (type solid)) (layer "F.CrtYd"))
-    (fp_line (start -1.95 -3.35) (end -0.95 -4.35)
-      (stroke (width 0.15) (type solid)) (layer "F.Fab"))
-    (fp_line (start -1.95 4.35) (end -1.95 -3.35)
-      (stroke (width 0.15) (type solid)) (layer "F.Fab"))
-    (fp_line (start -0.95 -4.35) (end 1.95 -4.35)
-      (stroke (width 0.15) (type solid)) (layer "F.Fab"))
-    (fp_line (start 1.95 -4.35) (end 1.95 4.35)
-      (stroke (width 0.15) (type solid)) (layer "F.Fab"))
-    (fp_line (start 1.95 4.35) (end -1.95 4.35)
-      (stroke (width 0.15) (type solid)) (layer "F.Fab"))
-    (pad "1" smd rect (at -2.6 -3.4925) (size 1.2 0.4) (layers "F.Cu" "F.Paste" "F.Mask")
-      (net 1 "unconnected-(U1-GND-Pad1)") (pinfunction "GND") (pintype "power_in"))
-    (pad "2" smd rect (at -2.6 -2.8575) (size 1.2 0.4) (layers "F.Cu" "F.Paste" "F.Mask")
-      (net 2 "unconnected-(U1-DIN-Pad2)") (pinfunction "DIN") (pintype "input"))
-    (pad "3" smd rect (at -2.6 -2.2225) (size 1.2 0.4) (layers "F.Cu" "F.Paste" "F.Mask")
-      (net 3 "unconnected-(U1-CLOCK-Pad3)") (pinfunction "CLOCK") (pintype "input"))
-    (pad "4" smd rect (at -2.6 -1.5875) (size 1.2 0.4) (layers "F.Cu" "F.Paste" "F.Mask")
-      (net 4 "unconnected-(U1-LATCH-Pad4)") (pinfunction "LATCH") (pintype "input"))
-    (pad "5" smd rect (at -2.6 -0.9525) (size 1.2 0.4) (layers "F.Cu" "F.Paste" "F.Mask")
-      (net 5 "unconnected-(U1-OUT0-Pad5)") (pinfunction "OUT0") (pintype "output"))
-    (pad "6" smd rect (at -2.6 -0.3175) (size 1.2 0.4) (layers "F.Cu" "F.Paste" "F.Mask")
-      (net 6 "unconnected-(U1-OUT1-Pad6)") (pinfunction "OUT1") (pintype "output"))
-    (pad "7" smd rect (at -2.6 0.3175) (size 1.2 0.4) (layers "F.Cu" "F.Paste" "F.Mask")
-      (net 7 "unconnected-(U1-OUT2-Pad7)") (pinfunction "OUT2") (pintype "output"))
-    (pad "8" smd rect (at -2.6 0.9525) (size 1.2 0.4) (layers "F.Cu" "F.Paste" "F.Mask")
-      (net 8 "unconnected-(U1-OUT3-Pad8)") (pinfunction "OUT3") (pintype "output"))
-    (pad "9" smd rect (at -2.6 1.5875) (size 1.2 0.4) (layers "F.Cu" "F.Paste" "F.Mask")
-      (net 9 "unconnected-(U1-OUT4-Pad9)") (pinfunction "OUT4") (pintype "output"))
-    (pad "10" smd rect (at -2.6 2.2225) (size 1.2 0.4) (layers "F.Cu" "F.Paste" "F.Mask")
-      (net 10 "unconnected-(U1-OUT5-Pad10)") (pinfunction "OUT5") (pintype "output"))
-    (pad "11" smd rect (at -2.6 2.8575) (size 1.2 0.4) (layers "F.Cu" "F.Paste" "F.Mask")
-      (net 11 "unconnected-(U1-OUT6-Pad11)") (pinfunction "OUT6") (pintype "output"))
-    (pad "12" smd rect (at -2.6 3.4925) (size 1.2 0.4) (layers "F.Cu" "F.Paste" "F.Mask")
-      (net 12 "unconnected-(U1-OUT7-Pad12)") (pinfunction "OUT7") (pintype "output"))
-    (pad "13" smd rect (at 2.6 3.4925) (size 1.2 0.4) (layers "F.Cu" "F.Paste" "F.Mask")
-      (net 13 "unconnected-(U1-OUT8-Pad13)") (pinfunction "OUT8") (pintype "output"))
-    (pad "14" smd rect (at 2.6 2.8575) (size 1.2 0.4) (layers "F.Cu" "F.Paste" "F.Mask")
-      (net 14 "unconnected-(U1-OUT9-Pad14)") (pinfunction "OUT9") (pintype "output"))
-    (pad "15" smd rect (at 2.6 2.2225) (size 1.2 0.4) (layers "F.Cu" "F.Paste" "F.Mask")
-      (net 15 "unconnected-(U1-OUT10-Pad15)") (pinfunction "OUT10") (pintype "output"))
-    (pad "16" smd rect (at 2.6 1.5875) (size 1.2 0.4) (layers "F.Cu" "F.Paste" "F.Mask")
-      (net 16 "unconnected-(U1-OUT11-Pad16)") (pinfunction "OUT11") (pintype "output"))
-    (pad "17" smd rect (at 2.6 0.9525) (size 1.2 0.4) (layers "F.Cu" "F.Paste" "F.Mask")
-      (net 17 "unconnected-(U1-OUT12-Pad17)") (pinfunction "OUT12") (pintype "output"))
-    (pad "18" smd rect (at 2.6 0.3175) (size 1.2 0.4) (layers "F.Cu" "F.Paste" "F.Mask")
-      (net 18 "unconnected-(U1-OUT13-Pad18)") (pinfunction "OUT13") (pintype "output"))
-    (pad "19" smd rect (at 2.6 -0.3175) (size 1.2 0.4) (layers "F.Cu" "F.Paste" "F.Mask")
-      (net 19 "unconnected-(U1-OUT14-Pad19)") (pinfunction "OUT14") (pintype "output"))
-    (pad "20" smd rect (at 2.6 -0.9525) (size 1.2 0.4) (layers "F.Cu" "F.Paste" "F.Mask")
-      (net 20 "unconnected-(U1-OUT15-Pad20)") (pinfunction "OUT15") (pintype "output"))
-    (pad "21" smd rect (at 2.6 -1.5875) (size 1.2 0.4) (layers "F.Cu" "F.Paste" "F.Mask")
-      (net 21 "unconnected-(U1-~{EN}-Pad21)") (pinfunction "~{EN}") (pintype "input"))
-    (pad "22" smd rect (at 2.6 -2.2225) (size 1.2 0.4) (layers "F.Cu" "F.Paste" "F.Mask")
-      (net 22 "unconnected-(U1-DOUT-Pad22)") (pinfunction "DOUT") (pintype "output"))
-    (pad "23" smd rect (at 2.6 -2.8575) (size 1.2 0.4) (layers "F.Cu" "F.Paste" "F.Mask")
-      (net 23 "unconnected-(U1-REXT-Pad23)") (pinfunction "REXT") (pintype "input"))
-    (pad "24" smd rect (at 2.6 -3.4925) (size 1.2 0.4) (layers "F.Cu" "F.Paste" "F.Mask")
-      (net 24 "unconnected-(U1-VDD-Pad24)") (pinfunction "VDD") (pintype "power_in"))
-    (model "${KICAD6_3DMODEL_DIR}/Package_SO.3dshapes/SSOP-24_3.9x8.7mm_P0.635mm.wrl"
-      (offset (xyz 0 0 0))
-      (scale (xyz 1 1 1))
-      (rotate (xyz 0 0 0))
-    )
-  )
-  (gr_rect (start 85.725 68.58) (end 99.695 86.995)
-    (stroke (width 0.1) (type default)) (fill none) (layer "Edge.Cuts"))
 )
