File: sixDigitDisplay.kicad_sch (KiCad schematic)
At the start: 3 parts, among them U5 XL7219, U6 CL2832AW, U7 CL2832AW

Commit message: Update footprints
Parts:
- U6, U7: footprint (none) -> SimPanel:DICE_2381
Changed lines of the file:
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@@
       (effects (font (size 1.27 1.27)))
     )
-    (property "Footprint" "" (at 176.53 92.71 0)
+    (property "Footprint" "SimPanel:DICE_2381" (at 176.53 92.71 0)
       (effects (font (size 1.27 1.27)) hide)
     )
@@
       (effects (font (size 1.27 1.27)))
     )
-    (property "Footprint" "" (at 243.84 92.71 0)
+    (property "Footprint" "SimPanel:DICE_2381" (at 243.84 92.71 0)
       (effects (font (size 1.27 1.27)) hide)
     )
